Commit message: 补充 Fast-LIO/ICP 重定位、Go2 仿真与导航 bringup 剩余改动。
含 Mid360 机头描述与 Gazebo 仿真包、CHAMP 第三方、TF/重定位与 launch 更新。

Co-authored-by: Cursor <cursoragent@cursor.com>

File: go2_description/xacro/const.xacro (robot description, xacro)
@@ -39,6 +39,6 @@
     <xacro:property name="calf_offset_z" value="-0.213"/>
     <!-- joint limits -->
-    <xacro:property name="damping" value="0.0"/>
-    <xacro:property name="friction" value="0.0"/>
+    <xacro:property name="damping" value="0.01"/>
+    <xacro:property name="friction" value="0.2"/>
     <xacro:property name="hip_position_max" value="1.0472"/>
     <xacro:property name="hip_position_min" value="-1.0472"/>
@@ -100,3 +100,4 @@
     <!-- foot -->
     <xacro:property name="foot_mass" value="0.06"/>
+    <!-- 站立角已按腿写入 robot_*.xacro 的 xacro:leg stand_* 参数（见 walk-these-ways-go2） -->
 </robot>

File: go2_description/xacro/gazebo.xacro (robot description, xacro)
@@ -1,235 +1,189 @@
 <?xml version="1.0"?>
 <robot>
-    <!-- ros_control plugin -->
     <gazebo>
-        <plugin name="gazebo_ros_control" filename="libgazebo_ros_control.so">
-            <robotNamespace>/go2_gazebo</robotNamespace>
-            <robotSimType>gazebo_ros_control/DefaultRobotHWSim</robotSimType>
-        </plugin>
-    </gazebo>
-    <!-- Show the trajectory of trunk center. -->
-    <!--gazebo>
-        <plugin name="3dplot" filename="libLinkPlot3DPlugin.so">
-            <frequency>10</frequency>
-            <plot>
-                <link>base</link>
-                <pose>0 0 0 0 0 0</pose>
-                <material>Gazebo/Yellow</material>
-            </plot>
-        </plugin>
-    </gazebo-->
-    <!-- Show the trajectory of foot. You can add another trajectory about another foot. -->
-     <gazebo>
-        <plugin name="3dplot" filename="libLinkPlot3DPlugin.so">
-            <frequency>100</frequency>
-            <plot>
-                <link>FL_foot</link>
-                <pose>0 0 0 0 0 0</pose>
-            </plot>
-        </plugin>
+      <plugin name="p3d_base_controller" filename="libgazebo_ros_p3d.so">
+        <ros>
+            <remapping>odom:=odom/ground_truth</remapping>
+        </ros>
+        <body_name>base_link</body_name>
+        <frame_name>world</frame_name>
+        <update_rate>10.0</update_rate>
+        <xyz_offset>0 0 0</xyz_offset>
+        <rpy_offset>0 0 0</rpy_offset>
+        <gaussian_noise>0.01</gaussian_noise>
+    </plugin>
     </gazebo>
     <gazebo>
-        <plugin filename="libgazebo_ros_force.so" name="gazebo_ros_force">
-            <bodyName>trunk</bodyName>
-            <topicName>/apply_force/trunk</topicName>
-        </plugin>
+        <plugin filename="libgazebo_ros2_control.so" name="gazebo_ros2_control">
+        <parameters>$(find go2_description)/config/ros_control/ros_control_sim.yaml</parameters>
+      </plugin>
     </gazebo>
     <gazebo reference="imu_link">
-        <gravity>true</gravity>
         <sensor name="imu_sensor" type="imu">
             <always_on>true</always_on>
-            <update_rate>1000</update_rate>
-            <visualize>true</visualize>
-            <topic>__default_topic__</topic>
-            <plugin filename="libgazebo_ros_imu_sensor.so" name="imu_plugin">
-                <topicName>trunk_imu</topicName>
-                <bodyName>imu_link</bodyName>
-                <updateRateHZ>1000.0</updateRateHZ>
-                <gaussianNoise>0.0</gaussianNoise>
-                <xyzOffset>0 0 0</xyzOffset>
-                <rpyOffset>0 0 0</rpyOffset>
-                <frameName>imu_link</frameName>
+            <update_rate>100</update_rate>
+            <imu>
+            <angular_velocity>
+                <x>
+                <noise type="gaussian">
+                    <mean>0.0</mean>
+                    <stddev>2e-4</stddev>
+                </noise>
+                </x>
+                <y>
+                <noise type="gaussian">
+                    <mean>0.0</mean>
+                    <stddev>2e-4</stddev>
+                </noise>
+                </y>
+                <z>
+                <noise type="gaussian">
+                    <mean>0.0</mean>
+                    <stddev>2e-4</stddev>
+                </noise>
+                </z>
+            </angular_velocity>
+            <linear_acceleration>
+                <x>
+                <noise type="gaussian">
+                    <mean>0.0</mean>
+                    <stddev>1.7e-2</stddev>
+                </noise>
+                </x>
+                <y>
+                <noise type="gaussian">
+                    <mean>0.0</mean>
+                    <stddev>1.7e-2</stddev>
+                </noise>
+                </y>
+                <z>
+                <noise type="gaussian">
+                    <mean>0.0</mean>
+                    <stddev>1.7e-2</stddev>
+                </noise>
+                </z>
+            </linear_acceleration>
+            </imu>
+            <plugin name="imu_plugin" filename="libgazebo_ros_imu_sensor.so">
+                <ros>
+                    <namespace>imu</namespace>
+                    <remapping>~/out:=data</remapping>
+                </ros>
+                <initial_orientation_as_reference>false</initial_orientation_as_reference>
             </plugin>
-            <pose>0 0 0 0 0 0</pose>
         </sensor>
     </gazebo>
-    <!-- Foot contacts. -->
-    <gazebo reference="FR_calf">
-        <sensor name="FR_foot_contact" type="contact">
-        <update_rate>100</update_rate>
-        <plugin name="contactPlugin" filename="libunitreeFootContactPlugin.so"/>
-        <contact>
-            <collision>FR_calf_fixed_joint_lump__FR_foot_collision_1</collision>
-        </contact>
-        </sensor>
-    </gazebo>
-    <gazebo reference="FL_calf">
-        <sensor name="FL_foot_contact" type="contact">
-        <update_rate>100</update_rate>
-        <plugin name="contactPlugin" filename="libunitreeFootContactPlugin.so"/>
-        <contact>
-            <collision>FL_calf_fixed_joint_lump__FL_foot_collision_1</collision>
-        </contact>
-        </sensor>
-    </gazebo>
-    <gazebo reference="RR_calf">
-        <sensor name="RR_foot_contact" type="contact">
-        <update_rate>100</update_rate>
-        <plugin name="contactPlugin" filename="libunitreeFootContactPlugin.so"/>
-        <contact>
-            <collision>RR_calf_fixed_joint_lump__RR_foot_collision_1</collision>
-        </contact>
-        </sensor>
-    </gazebo>
-    <gazebo reference="RL_calf">
-        <sensor name="RL_foot_contact" type="contact">
-        <update_rate>100</update_rate>
-        <plugin name="contactPlugin" filename="libunitreeFootContactPlugin.so"/>
-        <contact>
-            <collision>RL_calf_fixed_joint_lump__RL_foot_collision_1</collision>
-        </contact>
-        </sensor>
-    </gazebo>
-    <!-- Visualization of Foot contacts. -->
-    <gazebo reference="FR_foot">
-        <visual>
-            <plugin name="drawForcePlugin" filename="libunitreeDrawForcePlugin.so">
-                <topicName>FR_foot_contact</topicName>
-            </plugin>
-        </visual>
-    </gazebo>
-    <gazebo reference="FL_foot">
-        <visual>
-            <plugin name="drawForcePlugin" filename="libunitreeDrawForcePlugin.so">
-                <topicName>FL_foot_contact</topicName>
-            </plugin>
-        </visual>
-    </gazebo>
-    <gazebo reference="RR_foot">
-        <visual>
-            <plugin name="drawForcePlugin" filename="libunitreeDrawForcePlugin.so">
-                <topicName>RR_foot_contact</topicName>
-            </plugin>
-        </visual>
-    </gazebo>
-    <gazebo reference="RL_foot">
-        <visual>
-            <plugin name="drawForcePlugin" filename="libunitreeDrawForcePlugin.so">
-                <topicName>RL_foot_contact</topicName>
-            </plugin>
-        </visual>
-    </gazebo>
-    <gazebo reference="base">
+    <!-- <gazebo reference="base_link">
         <turnGravityOff>false</turnGravityOff>
-    </gazebo>
+    </gazebo> -->
     <gazebo reference="trunk">
         <mu1>0.2</mu1>
         <mu2>0.2</mu2>
-        <kp  value="1000000.0"/>
-        <kd  value="1.0"/>
+        <kp>10000.0</kp>
+        <kd>1.0</kd>
     </gazebo>
-    <gazebo reference="stick_link">
+    <!-- <gazebo reference="stick_link">
+        <mu1>0.2</mu1>
+        <mu2>0.2</mu2>
+    </gazebo> -->
+    <!-- <gazebo reference="imu_link">
+        <mu1>0.2</mu1>
+        <mu2>0.2</mu2>
+    </gazebo> -->
+    <!-- FL leg -->
+    <gazebo reference="lf_hip_link">
         <mu1>0.2</mu1>
         <mu2>0.2</mu2>
     </gazebo>
-    <gazebo reference="imu_link">
-        <mu1>0.2</mu1>
-        <mu2>0.2</mu2>
-    </gazebo>
-    <!-- FL leg -->
-    <gazebo reference="FL_hip">
-        <mu1>0.2</mu1>
-        <mu2>0.2</mu2>
-    </gazebo>
-    <gazebo reference="FL_thigh">
+    <gazebo reference="lf_upper_leg_link">
         <mu1>0.2</mu1>
         <mu2>0.2</mu2>
         <self_collide>1</self_collide>
-        <kp  value="1000000.0"/>
-        <kd  value="1.0"/>
+        <kp>10000.0</kp>
+        <kd>1.0</kd>
     </gazebo>
-    <gazebo reference="FL_calf">
+    <gazebo reference="lf_lower_leg_link">
         <mu1>0.2</mu1>
         <mu2>0.2</mu2>
         <self_collide>1</self_collide>
     </gazebo>
-    <gazebo reference="FL_foot">
+    <gazebo reference="lf_foot_link">
         <mu1>0.6</mu1>
         <mu2>0.6</mu2>
         <self_collide>1</self_collide>
-        <kp  value="1000000.0"/>
-        <kd  value="1.0"/>
+        <kp>10000.0</kp>
+        <kd>1.0</kd>
     </gazebo>
     <!-- FR leg -->
-    <gazebo reference="FR_hip">
+    <gazebo reference="rf_hip">
         <mu1>0.2</mu1>
         <mu2>0.2</mu2>
     </gazebo>
-    <gazebo reference="FR_thigh">
+    <gazebo reference="rf_upper_leg_link">
         <mu1>0.2</mu1>
         <mu2>0.2</mu2>
         <self_collide>1</self_collide>
-        <kp  value="1000000.0"/>
-        <kd  value="1.0"/>
+        <kp>10000.0</kp>
+        <kd>1.0</kd>
     </gazebo>
-    <gazebo reference="FR_calf">
+    <gazebo reference="rf_lower_leg_link">
         <mu1>0.2</mu1>
         <mu2>0.2</mu2>
         <self_collide>1</self_collide>
     </gazebo>
-    <gazebo reference="FR_foot">
+    <gazebo reference="rf_foot_link">
         <mu1>0.6</mu1>
         <mu2>0.6</mu2>
         <self_collide>1</self_collide>
-        <kp  value="1000000.0"/>
-        <kd  value="1.0"/>
+        <kp>10000.0</kp>
+        <kd>1.0</kd>
     </gazebo>
     <!-- RL leg -->
-    <gazebo reference="RL_hip">
+    <gazebo reference="lh_hip">
         <mu1>0.2</mu1>
         <mu2>0.2</mu2>
     </gazebo>
-    <gazebo reference="RL_thigh">
+    <gazebo reference="lh_upper_leg_link">
         <mu1>0.2</mu1>
         <mu2>0.2</mu2>
         <self_collide>1</self_collide>
-        <kp  value="1000000.0"/>
-        <kd  value="1.0"/>
+        <kp>10000.0</kp>
+        <kd>1.0</kd>
     </gazebo>
-    <gazebo reference="RL_calf">
+    <gazebo reference="lh_lower_leg_link">
         <mu1>0.2</mu1>
         <mu2>0.2</mu2>
         <self_collide>1</self_collide>
     </gazebo>
-    <gazebo reference="RL_foot">
+    <gazebo reference="lh_foot_link">
         <mu1>0.6</mu1>
         <mu2>0.6</mu2>
         <self_collide>1</self_collide>
-        <kp  value="1000000.0"/>
-        <kd  value="1.0"/>
+        <kp>10000.0</kp>
+        <kd>1.0</kd>
     </gazebo>
     <!-- RR leg -->
-    <gazebo reference="RR_hip">
+    <gazebo reference="rh_hip">
         <mu1>0.2</mu1>
         <mu2>0.2</mu2>
     </gazebo>
-    <gazebo reference="RR_thigh">
+    <gazebo reference="rh_upper_leg_link">
         <mu1>0.2</mu1>
         <mu2>0.2</mu2>
         <self_collide>1</self_collide>
-        <kp  value="1000000.0"/>
-        <kd  value="1.0"/>
+        <kp>10000.0</kp>
+        <kd>1.0</kd>
     </gazebo>
-    <gazebo reference="RR_calf">
+    <gazebo reference="rh_lower_leg_link">
         <mu1>0.2</mu1>
         <mu2>0.2</mu2>
         <self_collide>1</self_collide>
     </gazebo>
-    <gazebo reference="RR_foot">
+    <gazebo reference="rh_foot_link">
         <mu1>0.6</mu1>
         <mu2>0.6</mu2>
         <self_collide>1</self_collide>
-        <kp  value="1000000.0"/>
-        <kd  value="1.0"/>
+        <kp>10000.0</kp>
+        <kd>1.0</kd>
     </gazebo>
 </robot>

File: go2_description/xacro/leg.xacro (robot description, xacro)
@@ -1,6 +1,6 @@
 <?xml version="1.0"?>
 <robot xmlns:xacro="http://www.ros.org/wiki/xacro">
-    <xacro:include filename="$(find go2_description)/xacro/transmission.xacro"/>
-    <xacro:macro name="leg" params="name mirror mirror_dae front_hind front_hind_dae">
+    <!-- <xacro:include filename="$(find go2_description)/xacro/transmission.xacro"/> -->
+    <xacro:macro name="leg" params="name mirror mirror_dae front_hind front_hind_dae stand_hip:=0.0 stand_thigh:=0.8 stand_calf:=-1.5">
         <joint name="${name}_hip_joint" type="revolute">
             <xacro:if value="${(mirror_dae == False) and (front_hind_dae == True)}">
@@ -17,5 +17,5 @@
             </xacro:if>
             <parent link="trunk"/>
-            <child link="${name}_hip"/>
+            <child link="${name}_hip_link"/>
             <axis xyz="1 0 0"/>
             <dynamics damping="${damping}" friction="${friction}"/>
@@ -27,5 +27,5 @@
             </xacro:if>
         </joint>
-        <link name="${name}_hip">
+        <link name="${name}_hip_link">
             <visual>
                 <xacro:if value="${(mirror_dae == True) and (front_hind_dae == True)}">
@@ -42,5 +42,5 @@
                 </xacro:if>
                 <geometry>
-                    <mesh filename="package://go2_description/meshes/hip.dae" scale="1 1 1"/>
+                    <mesh filename="file://$(find go2_description)/meshes/hip.dae" scale="1 1 1"/>
                 </geometry>
                 <!-- <material name="orange"/> -->
@@ -61,21 +61,21 @@
             </inertial>
         </link>
-        <joint name="${name}_thigh_joint" type="revolute">
+        <joint name="${name}_upper_leg_joint" type="revolute">
             <origin rpy="0 0 0" xyz="0 ${thigh_offset*mirror} 0"/>
-            <parent link="${name}_hip"/>
-            <child link="${name}_thigh"/>
+            <parent link="${name}_hip_link"/>
+            <child link="${name}_upper_leg_link"/>
             <axis xyz="0 1 0"/>
             <dynamics damping="${damping}" friction="${friction}"/>
             <limit effort="${thigh_torque_max}" velocity="${thigh_velocity_max}" lower="${thigh_position_min}" upper="${thigh_position_max}"/>
         </joint>
-        <link name="${name}_thigh">
+        <link name="${name}_upper_leg_link">
             <visual>
                 <origin rpy="0 0 0" xyz="0 0 0"/>
                 <geometry>
                     <xacro:if value="${mirror_dae == True}">
-                        <mesh filename="package://go2_description/meshes/thigh.dae" scale="1 1 1"/>
+                        <mesh filename="file://$(find go2_description)/meshes/thigh.dae" scale="1 1 1"/>
                     </xacro:if>
                     <xacro:if value="${mirror_dae == False}">
-                        <mesh filename="package://go2_description/meshes/thigh_mirror.dae" scale="1 1 1"/>
+                        <mesh filename="file://$(find go2_description)/meshes/thigh_mirror.dae" scale="1 1 1"/>
                     </xacro:if>
                 </geometry>
@@ -97,17 +97,17 @@
             </inertial>
         </link>
-        <joint name="${name}_calf_joint" type="revolute">
+        <joint name="${name}_lower_leg_joint" type="revolute">
             <origin rpy="0 0 0" xyz="0 0 ${-thigh_length}"/>
-            <parent link="${name}_thigh"/>
-            <child link="${name}_calf"/>
+            <parent link="${name}_upper_leg_link"/>
+            <child link="${name}_lower_leg_link"/>
             <axis xyz="0 1 0"/>
             <dynamics damping="${damping}" friction="${friction}"/>
             <limit effort="${calf_torque_max}" velocity="${calf_velocity_max}" lower="${calf_position_min}" upper="${calf_position_max}"/>
         </joint>
-        <link name="${name}_calf">
+        <link name="${name}_lower_leg_link">
             <visual>
                 <origin rpy="0 0 0" xyz="0 0 0"/>
                 <geometry>
-                    <mesh filename="package://go2_description/meshes/calf.dae" scale="1 1 1"/>
+                    <mesh filename="file://$(find go2_description)/meshes/calf.dae" scale="1 1 1"/>
                 </geometry>
                 <!-- <material name="orange"/> -->
@@ -128,10 +128,10 @@
             </inertial>
         </link>
-        <joint name="${name}_foot_fixed" type="fixed">0
+        <joint name="${name}_foot_joint" type="fixed">0
             <origin rpy="0 0 0" xyz="0 0 ${-(calf_length)}"/>
-            <parent link="${name}_calf"/>
-            <child link="${name}_foot"/>
+            <parent link="${name}_lower_leg_link"/>
+            <child link="${name}_foot_link"/>
         </joint>
-        <link name="${name}_foot">
+        <link name="${name}_foot_link">
             <visual>
                 <origin rpy="0 0 0" xyz="0 0 0"/>
@@ -155,5 +155,28 @@
             </inertial>
         </link>
-        <xacro:leg_transmission name="${name}"/>
+        <ros2_control name="${name}" type="system">
+            <hardware>
+                <plugin>gazebo_ros2_control/GazeboSystem</plugin>
+            </hardware>
+            <joint name="${name}_hip_joint">
+                <command_interface name="effort"/>
+                <state_interface name="position"/>
+                <state_interface name="velocity"/>
+                <param name="initial_value">${stand_hip}</param>
+            </joint>
+            <joint name="${name}_upper_leg_joint">
+                <command_interface name="effort"/>
+                <state_interface name="position"/>
+                <state_interface name="velocity"/>
+                <param name="initial_value">${stand_thigh}</param>
+            </joint>
+            <joint name="${name}_lower_leg_joint">
+                <command_interface name="effort"/>
+                <state_interface name="position"/>
+                <state_interface name="velocity"/>
+                <param name="initial_value">${stand_calf}</param>
+            </joint>
+        </ros2_control>
+        <!-- <xacro:leg_transmission name="${name}"/> -->
     </xacro:macro>
 </robot>

File: go2_description/xacro/robot.xacro (robot description, xacro)
@@ -17,8 +17,8 @@
             <origin rpy="0 0 0" xyz="0 0 0"/>
             <parent link="world"/>
-            <child link="base"/>
+            <child link="base_link"/>
         </joint>
     </xacro:if>
-    <link name="base">
+    <link name="base_link">
         <visual>
             <origin rpy="0 0 0" xyz="0 0 0"/>
@@ -30,5 +30,5 @@
     <joint name="floating_base" type="fixed">
         <origin rpy="0 0 0" xyz="0 0 0"/>
-        <parent link="base"/>
+        <parent link="base_link"/>
         <child link="trunk"/>
     </joint>
@@ -37,5 +37,5 @@
             <origin rpy="0 0 0" xyz="0 0 0"/>
             <geometry>
-                <mesh filename="package://go2_description/meshes/trunk.dae" scale="1 1 1"/>
+                <mesh filename="file://$(find go2_description)/meshes/trunk.dae" scale="1 1 1"/>
             </geometry>
             <!-- <material name="orange"/> -->
@@ -72,5 +72,4 @@
                 <box size="0.001 0.001 0.001"/>
             </geometry>
-            <!-- <material name="red"/> -->
         </visual>
         <collision>
@@ -107,7 +106,7 @@
     </link>
 -->
-    <xacro:leg name="FR" mirror="-1" mirror_dae= "False" front_hind="1"  front_hind_dae="True"  />
-    <xacro:leg name="FL" mirror="1"  mirror_dae="True"   front_hind="1"  front_hind_dae="True"  />
-    <xacro:leg name="RR" mirror="-1" mirror_dae="False"  front_hind="-1" front_hind_dae="False" />
-    <xacro:leg name="RL" mirror="1"  mirror_dae="True"   front_hind="-1" front_hind_dae="False" />
+    <xacro:leg name="rf" mirror="-1" mirror_dae="False" front_hind="1"  front_hind_dae="True"  stand_hip="-0.1" stand_thigh="0.8" stand_calf="-1.5"/>
+    <xacro:leg name="lf" mirror="1"  mirror_dae="True"   front_hind="1"  front_hind_dae="True"  stand_hip="0.1"  stand_thigh="0.8" stand_calf="-1.5"/>
+    <xacro:leg name="rh" mirror="-1" mirror_dae="False" front_hind="-1" front_hind_dae="False" stand_hip="-0.1" stand_thigh="1.0" stand_calf="-1.5"/>
+    <xacro:leg name="lh" mirror="1"  mirror_dae="True"   front_hind="-1" front_hind_dae="False" stand_hip="0.1"  stand_thigh="1.0" stand_calf="-1.5"/>
 </robot>

File: go2_description/xacro/transmission.xacro (robot description, xacro)
@@ -12,20 +12,20 @@
             </actuator>
         </transmission>
-        <transmission name="${name}_thigh_tran">
+        <transmission name="${name}_upper_leg_tran">
             <type>transmission_interface/SimpleTransmission</type>
-            <joint name="${name}_thigh_joint">
+            <joint name="${name}_upper_leg_joint">
             <hardwareInterface>hardware_interface/EffortJointInterface</hardwareInterface>
             </joint>
-            <actuator name="${name}_thigh_motor">
+            <actuator name="${name}_upper_leg_motor">
             <hardwareInterface>hardware_interface/EffortJointInterface</hardwareInterface>
             <mechanicalReduction>1</mechanicalReduction>
             </actuator>
         </transmission>
-        <transmission name="${name}_calf_tran">
+        <transmission name="${name}_lower_leg_tran">
             <type>transmission_interface/SimpleTransmission</type>
-            <joint name="${name}_calf_joint">
+            <joint name="${name}_lower_leg_joint">
             <hardwareInterface>hardware_interface/EffortJointInterface</hardwareInterface>
             </joint>
-            <actuator name="${name}_calf_motor">
+            <actuator name="${name}_lower_leg_motor">
             <hardwareInterface>hardware_interface/EffortJointInterface</hardwareInterface>
             <mechanicalReduction>1</mechanicalReduction>
