Commit message: 增强 Go2 EGO 局部避障与四足导航控制，并整理仿真模型栈。
改进 EGO 重规划与栅格地图同步、轨迹前瞻跟踪和四足动力学参数，提升转弯与绕障能力；同时更新 go2_description/champ 仿真集成与重定位相关配置。

Co-authored-by: Cursor <cursoragent@cursor.com>

File: go2_description/urdf/go2_description.urdf (robot description, URDF)
Before this commit: robot go2_description, 29 links, 28 joints
Links:
- added link base, mass 6.921; collision box size=0.3762 0.0935 0.114; visual mesh filename=file://$(find go2_description)/dae/base.dae
- link FL_calf: geometry collision cylinder length=0.12 radius=0.012; visual mesh filename=file://$(find go2_description)/dae/calf.obj
- link FL_foot: geometry collision sphere radius=0.022; visual mesh filename=file://$(find go2_description)/dae/foot.dae
- link FL_hip: geometry collision cylinder length=0.04 radius=0.046; visual mesh filename=file://$(find go2_description)/dae/hip.dae
- link FL_thigh: geometry collision box size=0.213 0.0245 0.034; visual mesh filename=file://$(find go2_description)/dae/thigh.dae
- link FR_calf: geometry collision cylinder length=0.12 radius=0.013; visual mesh filename=file://$(find go2_description)/dae/calf_mirror.dae
- link FR_foot: geometry collision sphere radius=0.022; visual mesh filename=file://$(find go2_description)/dae/foot.dae
- link FR_hip: geometry collision cylinder length=0.04 radius=0.046; visual mesh filename=file://$(find go2_description)/dae/hip.dae
- link FR_thigh: geometry collision box size=0.213 0.0245 0.034; visual mesh filename=file://$(find go2_description)/dae/thigh_mirror.dae
- link RL_calf: geometry collision cylinder length=0.12 radius=0.013; visual mesh filename=file://$(find go2_description)/dae/calf.obj
- link RL_foot: geometry collision sphere radius=0.022; visual mesh filename=file://$(find go2_description)/dae/foot.dae
- link RL_hip: geometry collision cylinder length=0.04 radius=0.046; visual mesh filename=file://$(find go2_description)/dae/hip.dae
- link RL_thigh: geometry collision box size=0.213 0.0245 0.034; visual mesh filename=file://$(find go2_description)/dae/thigh.dae
- link RR_calf: geometry collision cylinder length=0.12 radius=0.013; visual mesh filename=file://$(find go2_description)/dae/calf_mirror.dae
- link RR_foot: geometry collision sphere radius=0.022; visual mesh filename=file://$(find go2_description)/dae/foot.dae
- link RR_hip: geometry collision cylinder length=0.04 radius=0.046; visual mesh filename=file://$(find go2_description)/dae/hip.dae
- link RR_thigh: geometry collision box size=0.213 0.0245 0.034; visual mesh filename=file://$(find go2_description)/dae/thigh_mirror.dae
- link base_link: mass 6.921 -> None; geometry 
Joints:
- added joint base_joint: type fixed, parent base_link, child base, origin xyz=0 0 0 rpy=0 0 0
- joint FL_hip_joint: parent base_link -> base
- joint FR_hip_joint: parent base_link -> base
- joint Head_upper_joint: parent base_link -> base
- joint RL_hip_joint: parent base_link -> base
- joint RR_hip_joint: parent base_link -> base
- joint imu_joint: parent base_link -> base
- joint radar_joint: parent base_link -> base

File: go2_description/xacro/const.xacro (robot description, xacro)
@@ -1,4 +1,4 @@
 <?xml version="1.0"?>
-<robot xmlns:xacro="http://www.ros.org/wiki/xacro">
+<robot name="go2" xmlns:xacro="http://www.ros.org/wiki/xacro">
     <!-- Constants for robot dimensions -->
     <xacro:property name="PI" value="3.1415926535897931"/>
@@ -39,65 +39,92 @@
     <xacro:property name="calf_offset_z" value="-0.213"/>
     <!-- joint limits -->
-    <xacro:property name="damping" value="0.01"/>
-    <xacro:property name="friction" value="0.2"/>
+    <xacro:property name="damping" value="0.5"/>
+    <xacro:property name="friction" value="0.5"/>
     <xacro:property name="hip_position_max" value="1.0472"/>
     <xacro:property name="hip_position_min" value="-1.0472"/>
-    <xacro:property name="hip_velocity_max" value="30.1"/>
+    <xacro:property name="hip_velocity_max" value="1.5"/>
+    <!-- <xacro:property name="hip_velocity_max" value="30.1"/> -->
     <xacro:property name="hip_torque_max" value="23.7"/>
     <xacro:property name="thigh_position_max" value="3.4907"/>
     <xacro:property name="thigh_position_min" value="-1.5708"/>
-    <xacro:property name="thigh_velocity_max" value="30.1"/>
+    <xacro:property name="thigh_velocity_max" value="1.5"/>
+    <!-- <xacro:property name="thigh_velocity_max" value="30.1"/> -->
     <xacro:property name="thigh_torque_max" value="23.7"/>
     <xacro:property name="calf_position_max" value="-0.83776"/>
     <xacro:property name="calf_position_min" value="-2.7227"/>
-    <xacro:property name="calf_velocity_max" value="20.06"/>
-    <xacro:property name="calf_torque_max" value="35.55"/>
+    <xacro:property name="calf_velocity_max" value="1.5"/>
+    <!-- <xacro:property name="calf_velocity_max" value="20.06"/> -->
+    <!-- <xacro:property name="calf_torque_max" value="35.55"/> -->
+    <xacro:property name="calf_torque_max" value="25"/>
     <!-- dynamics inertial value -->
     <!-- trunk -->
     <xacro:property name="trunk_mass" value="6.921"/>
+    <!-- <xacro:property name="trunk_mass" value="6.921"/> -->
+    <!-- <xacro:property name="trunk_mass" value="2"/> -->
     <xacro:property name="trunk_com_x" value="0.021112"/>
     <xacro:property name="trunk_com_y" value="0.00"/>
     <xacro:property name="trunk_com_z" value="-0.005366"/>
-    <xacro:property name="trunk_ixx" value="0.02448"/>
+    <xacro:property name="trunk_ixx" value="0.01683"/>
+    <xacro:property name="trunk_ixy" value="0.0"/>
+    <xacro:property name="trunk_ixz" value="0.0"/>
+    <xacro:property name="trunk_iyy" value="0.044483"/>
+    <xacro:property name="trunk_iyz" value="0"/>
+    <xacro:property name="trunk_izz" value="0.055683"/>
+    <!-- <xacro:property name="trunk_ixx" value="0.02448"/>
     <xacro:property name="trunk_ixy" value="0.00012166"/>
     <xacro:property name="trunk_ixz" value="0.0014849"/>
     <xacro:property name="trunk_iyy" value="0.098077"/>
     <xacro:property name="trunk_iyz" value="-3.12E-05"/>
-    <xacro:property name="trunk_izz" value="0.107"/>
+    <xacro:property name="trunk_izz" value="0.107"/> -->
     <!-- hip (left front) -->
     <xacro:property name="hip_mass" value="0.678"/>
+    <!-- <xacro:property name="hip_mass" value="0.250"/> -->
     <xacro:property name="hip_com_x" value="-0.0054"/>
     <xacro:property name="hip_com_y" value="0.00194"/>
     <xacro:property name="hip_com_z" value="-0.000105"/>
     <xacro:property name="hip_ixx" value="0.00048"/>
-    <xacro:property name="hip_ixy" value="-3.01E-06"/>
-    <xacro:property name="hip_ixz" value="1.11E-06"/>
+    <xacro:property name="hip_ixy" value="0.0"/>
+    <!-- <xacro:property name="hip_ixy" value="-3.01E-06"/> -->
+    <xacro:property name="hip_ixz" value="0.0"/>
+    <!-- <xacro:property name="hip_ixz" value="1.11E-06"/> -->
     <xacro:property name="hip_iyy" value="0.000884"/>
-    <xacro:property name="hip_iyz" value="-1.42E-06"/>
+    <xacro:property name="hip_iyz" value="0.0"/>
+    <!-- <xacro:property name="hip_iyz" value="-1.42E-06"/> -->
     <xacro:property name="hip_izz" value="0.000596"/>
     <!-- thigh -->
-    <xacro:property name="thigh_mass" value="1.152"/>
+    <!-- <xacro:property name="thigh_mass" value="1.152"/> -->
+    <xacro:property name="thigh_mass" value="0.552"/>
+    <!-- <xacro:property name="thigh_mass" value="0.125"/> -->
     <xacro:property name="thigh_com_x" value="-0.00374"/>
     <xacro:property name="thigh_com_y" value="-0.0223"/>
     <xacro:property name="thigh_com_z" value="-0.0327"/>
     <xacro:property name="thigh_ixx" value="0.00584"/>
-    <xacro:property name="thigh_ixy" value="8.72E-05"/>
-    <xacro:property name="thigh_ixz" value="-0.000289"/>
-    <xacro:property name="thigh_iyy" value="0.0058"/>
-    <xacro:property name="thigh_iyz" value="0.000808"/>
-    <xacro:property name="thigh_izz" value="0.00103"/>
+    <!-- <xacro:property name="thigh_ixx" value="0.00584"/> -->
+    <xacro:property name="thigh_ixy" value="0.0"/>
+    <!-- <xacro:property name="thigh_ixy" value="8.72E-05"/> -->
+    <xacro:property name="thigh_ixz" value="-0.0"/>
+    <!-- <xacro:property name="thigh_ixz" value="-0.000289"/> -->
+    <xacro:property name="thigh_iyy" value="0.0011"/>
+    <!-- <xacro:property name="thigh_iyy" value="0.0058"/> -->
+    <xacro:property name="thigh_iyz" value="0.0"/>
+    <!-- <xacro:property name="thigh_iyz" value="0.000808"/> -->
+    <xacro:property name="thigh_izz" value="3.29E-05"/>
+    <!-- <xacro:property name="thigh_izz" value="0.00103"/> -->
     <!-- calf -->
-    <xacro:property name="calf_mass" value="0.154"/>
+    <!-- <xacro:property name="calf_mass" value="0.154"/> -->
+    <xacro:property name="calf_mass" value="0.125"/>
     <xacro:property name="calf_com_x" value="0.00548"/>
     <xacro:property name="calf_com_y" value="-0.000975"/>
     <xacro:property name="calf_com_z" value="-0.115"/>
     <xacro:property name="calf_ixx" value="0.00108"/>
-    <xacro:property name="calf_ixy" value="3.4E-07"/>
-    <xacro:property name="calf_ixz" value="1.72E-05"/>
+    <xacro:property name="calf_ixy" value="0"/>
+    <!-- <xacro:property name="calf_ixy" value="3.4E-07"/> -->
+    <xacro:property name="calf_ixz" value="0"/>
+    <!-- <xacro:property name="calf_ixz" value="1.72E-05"/> -->
     <xacro:property name="calf_iyy" value="0.0011"/>
-    <xacro:property name="calf_iyz" value="8.28E-06"/>
+    <xacro:property name="calf_iyz" value="0"/>
+    <!-- <xacro:property name="calf_iyz" value="8.28E-06"/> -->
     <xacro:property name="calf_izz" value="3.29E-05"/>
     <!-- foot -->
-    <xacro:property name="foot_mass" value="0.06"/>
-    <!-- 站立角已按腿写入 robot_*.xacro 的 xacro:leg stand_* 参数（见 walk-these-ways-go2） -->
+    <xacro:property name="foot_mass" value="0.006"/>
 </robot>

File: go2_description/xacro/robot_mid360.xacro (robot description, xacro)
@@ -1,10 +1,15 @@
 <?xml version="1.0"?>
 <robot name="go2_mid360" xmlns:xacro="http://www.ros.org/wiki/xacro">
-    <xacro:arg name="DEBUG" default="false"/>
+    <!-- <xacro:arg name="DEBUG" default="false"/> -->
     <xacro:include filename="$(find go2_description)/xacro/const.xacro"/>
     <xacro:include filename="$(find go2_description)/xacro/materials.xacro"/>
-    <xacro:include filename="$(find go2_description)/xacro/leg.xacro"/>
+    <xacro:include filename="$(find go2_description)/xacro/go2_leg.xacro"/>
+    <!-- <xacro:include filename="/home/e-yantra/unitree_ws/install/go2_description/share/go2_description/xacro/const.xacro"/>
+    <xacro:include filename="/home/e-yantra/unitree_ws/install/go2_description/share/go2_description/xacro/materials.xacro"/>
+    <xacro:include filename="/home/e-yantra/unitree_ws/install/go2_description/share/go2_description/xacro/leg.xacro"/> -->
+    <!-- <xacro:include filename="/home/e-yantra/unitree_ws/install/go2_description/share/go2_description/xacro/leg.xacro"/> -->
+    <!-- find-pkg-share -->
     <!-- <xacro:include filename="$(find go2_description)/xacro/stairs.xacro"/> -->
-    <xacro:include filename="$(find go2_description)/xacro/gazebo.xacro"/>
+    <!-- <xacro:include filename="$(find go2_description)/urdf/gazebo.xacro"/> -->
     <!-- <xacro:include filename="$(find go2_gazebo)/launch/stairs.urdf.xacro"/> -->
     <!-- <xacro:stairs stairs="15" xpos="0" ypos="0" zpos="0" /> -->
@@ -12,12 +17,14 @@
     <!-- Actually, the rotor will rotate and the joint is not fixed. Reduction ratio should be considered. -->
     <!-- Debug mode will hung up the robot, use "true" or "false" to switch it. -->
-    <xacro:if value="$(arg DEBUG)">
-        <link name="world"/>
-        <joint name="base_static_joint" type="fixed">
-            <origin rpy="0 0 0" xyz="0 0 0"/>
-            <parent link="world"/>
-            <child link="base_link"/>
-        </joint>
-    </xacro:if>
+    <!-- <xacro:if value="$(arg DEBUG)">
+    </xacro:if>  -->
+    <!-- <link name="world"/>
+    <link name="map"/>
+    <joint name="base_static_joint" type="fixed">
+        <origin rpy="0 0 0" xyz="0 0 0"/>
+        <parent link="world"/>
+        <child link="map"/>
+    </joint> -->
+    <xacro:include filename="$(find go2_description)/xacro/accessories_mid360.urdf.xacro" />
     <link name="base_link">
         <visual>
@@ -44,10 +51,17 @@
             <origin rpy="0 0 0" xyz="0 0 0"/>
             <geometry>
-                <box size="${trunk_length} ${trunk_width} ${trunk_height}"/>
+                <box size="0.3762 0.0935 0.114"/>
             </geometry>
         </collision>
         <inertial>
+            <!-- <origin rpy="0 0 0" xyz="0.021112 0 -0.005366"/> -->
             <origin rpy="0 0 0" xyz="${trunk_com_x} ${trunk_com_y} ${trunk_com_z}"/>
+            <!-- <mass value="6.921"/> -->
+            <!-- <mass value="2"/> -->
             <mass value="${trunk_mass}"/>
+            <!-- <inertia
+                ixx="0.02448" ixy="0.00012166" ixz="0.0014849"
+                iyy="0.098077" iyz="-3.12E-05"
+                izz="0.107"/>   -->
             <inertia
                 ixx="${trunk_ixx}" ixy="${trunk_ixy}" ixz="${trunk_ixz}"
@@ -56,5 +70,10 @@
         </inertial>
     </link>
-    <joint name="imu_joint" type="fixed">
+    <xacro:accessories_mid360
+        base_name="base_link"
+        base_length="0.3762"
+        base_height="0.114"
+    />
+    <!-- <joint name="imu_joint" type="fixed">
         <parent link="trunk"/>
         <child link="imu_link"/>
@@ -72,4 +91,5 @@
                 <box size="0.001 0.001 0.001"/>
             </geometry>
+            <material name="red"/>
         </visual>
         <collision>
@@ -79,5 +99,5 @@
             </geometry>
         </collision>
-    </link>
+    </link> -->
     <!--
     <joint name="load_joint" type="fixed">
@@ -106,10 +126,30 @@
     </link>
 -->
-    <!-- 站立角参考 walk-these-ways-go2 / 多数 Go2 仿真 URDF（前腿大腿 0.8，后腿 1.0，小腿 -1.5） -->
-    <xacro:leg name="rf" mirror="-1" mirror_dae="False" front_hind="1"  front_hind_dae="True"  stand_hip="-0.1" stand_thigh="0.8" stand_calf="-1.5"/>
-    <xacro:leg name="lf" mirror="1"  mirror_dae="True"   front_hind="1"  front_hind_dae="True"  stand_hip="0.1"  stand_thigh="0.8" stand_calf="-1.5"/>
-    <xacro:leg name="rh" mirror="-1" mirror_dae="False" front_hind="-1" front_hind_dae="False" stand_hip="-0.1" stand_thigh="1.0" stand_calf="-1.5"/>
-    <xacro:leg name="lh" mirror="1"  mirror_dae="True"   front_hind="-1" front_hind_dae="False" stand_hip="0.1"  stand_thigh="1.0" stand_calf="-1.5"/>
-  <!-- navmid360: 狗头 Mid-360；点云 pitch=19° 由 Gazebo 插件 extrinsic 与 MID360_config.json 一致 -->
+    <xacro:leg name="lf" mirror="1"  mirror_dae="True"   front_hind="1"  front_hind_dae="True"  />
+    <xacro:leg name="rf" mirror="-1" mirror_dae= "False" front_hind="1"  front_hind_dae="True"  />
+    <xacro:leg name="lh" mirror="1"  mirror_dae="True"   front_hind="-1" front_hind_dae="False" />
+    <xacro:leg name="rh" mirror="-1" mirror_dae="False"  front_hind="-1" front_hind_dae="False" />
+    <gazebo>
+      <plugin name="p3d_base_controller" filename="libgazebo_ros_p3d.so">
+        <ros>
+            <argument>odom:=odom/ground_truth</argument>
+        </ros>
+        <body_name>base_link</body_name>
+        <frame_name>world</frame_name>
+        <update_rate>10.0</update_rate>
+        <xyz_offset>0 0 0</xyz_offset>
+        <rpy_offset>0 0 0</rpy_offset>
+        <gaussian_noise>0.01</gaussian_noise>
+    </plugin>
+    </gazebo>
+    <gazebo>
+        <plugin filename="libgazebo_ros2_control.so" name="gazebo_ros2_control">
+            <!-- <parameters>$(find-pkg-share go2_description)/config/go2_controlgdsf.yaml</parameters> -->
+            <!-- <parameters>"${find go2_description}/config/go2_control.yaml"</parameters> -->
+            <parameters>$(find go2_description)/config/ros_control/ros_control_sim.yaml</parameters>
+            <!-- <parameters>/home/e-yantra/unitree_ws/install/go2_description/share/go2_description/config/go2_control.yaml</parameters> -->
+        </plugin>
+    </gazebo>
+  <!-- navmid360: 狗头 Mid-360；点云 pitch=19° 与 MID360_config.json 一致 -->
   <xacro:include filename="$(find go2_description)/xacro/mid360_head_mount.xacro"/>
   <xacro:go2_mid360_head_mount parent="trunk" topic="livox/lidar"/>
